Commit message: sent commands to position_trajectory_controller

File: schunk_description/ros2_control/schunk_lwa4p_mock_hardware.ros2_control.xacro (robot description, xacro)
@@ -1,5 +1,5 @@
 <?xml version="1.0"?>
 <robot xmlns:xacro="http://www.ros.org/wiki/xacro" name="6dof_robot">
-  <xacro:macro name="schunk_lwa4p_system_position_only" params="name prefix use_gazebo:=^|false use_mock_hardware:=^|true mock_sensor_commands:=^|false ">
+  <xacro:macro name="schunk_lwa4p_mock_hardware" params="name use_gazebo:=^|false use_mock_hardware:=^|true mock_sensor_commands:=^|false ">
     <ros2_control name="${name}" type="system">
       <xacro:if value="${use_gazebo}">
@@ -17,5 +17,5 @@
         </hardware>
       </xacro:unless>
-      <joint name="${prefix}_1_joint">
+      <joint name="${name}_1_joint">
         <command_interface name="position">
           <param name="min">-2.95</param>
@@ -24,5 +24,5 @@
         <state_interface name="position"/>
       </joint>
-      <joint name="${prefix}_2_joint">
+      <joint name="${name}_2_joint">
         <command_interface name="position">
           <param name="min">-2.95</param>
@@ -31,5 +31,5 @@
         <state_interface name="position"/>
       </joint>
-      <joint name="${prefix}_3_joint">
+      <joint name="${name}_3_joint">
         <command_interface name="position">
           <param name="min">-2.69</param>
@@ -38,5 +38,5 @@
         <state_interface name="position"/>
       </joint>
-      <joint name="${prefix}_4_joint">
+      <joint name="${name}_4_joint">
         <command_interface name="position">
           <param name="min">-2.95</param>
@@ -45,5 +45,5 @@
         <state_interface name="position"/>
       </joint>
-      <joint name="${prefix}_5_joint">
+      <joint name="${name}_5_joint">
         <command_interface name="position">
           <param name="min">-2.95</param>
@@ -52,5 +52,5 @@
         <state_interface name="position"/>
       </joint>
-      <joint name="${prefix}_6_joint">
+      <joint name="${name}_6_joint">
         <command_interface name="position">
           <param name="min">-2.95</param>

File: schunk_description/urdf/schunk_lwa4p.urdf.xacro (robot description, xacro)
@@ -18,5 +18,5 @@
   <xacro:include filename="$(find schunk_description)/urdf/materials.urdf.xacro" />
   <!-- Import RRBot ros2_control description -->
-  <xacro:include filename="$(find schunk_description)/ros2_control/schunk_lwa4p_system_position_only.ros2_control.xacro" />
+  <xacro:include filename="$(find schunk_description)/ros2_control/schunk_lwa4p_mock_hardware.ros2_control.xacro" />
   <!-- Used for fixing robot -->
   <link name="world"/>
@@ -27,6 +27,6 @@
     <origin xyz="0 0 0" rpy="0 0 0" />
   </xacro:schunk_lwa4p>
-  <xacro:schunk_lwa4p_system_position_only
-    name="SchunkLwa4pSystemPositionOnly" prefix="$(arg prefix)arm"
+  <xacro:schunk_lwa4p_mock_hardware
+    name="$(arg prefix)arm"
     use_mock_hardware="$(arg use_mock_hardware)"
     mock_sensor_commands="$(arg mock_sensor_commands)"
